File: Eagle.cad/EEPROM AT28C16 Helper.sch (EAGLE design)
At the start: 13 parts

Commit message: Some code and schematic
Parts:
- removed 28C16AP: 28C16AP, microchip:28C16AP
- removed CAP: (no value), pinhead:PINHD-1X2
- removed EEPROM_ADDR, EEPROM_DATA: PINHD-1X10, adafruit:PINHD-1X10
- removed JP_D13_VCC_GND, JP_DC11_DC10: (no value), adafruit:PINHD-1X15
- removed POWER_LED, WRITE_EN_LED: (no value), adafruit:LEDSMT1206
- removed R_POWER_LED, R_WRITE_EN_LED, R_WRITE_EN_PU: (no value), adafruit:R-US_R1206
- removed SR_0, SR_1: 74HC595N, 74xx-eu:74HC595N
- added 28C16A_EEPROM: 28C16AP, microchip:28C16AP
- added ADDRESS: (no value), pinhead:PINHD-1X11
- added CHIP_ENABLE_TO_GND: (no value), microbuilder:SOLDERJUMPERREFLOW
- added DATA: PINHD-1X10, adafruit:PINHD-1X10
- added ENABLE: (no value), adafruit:PINHD-1X3
- added R_PUP_2K: (no value), adafruit:R-US_R1206
Connections:
- removed net EEPROM_A0: 28C16AP.A0, EEPROM_ADDR.1, SR_0A.QA
- removed net EEPROM_A1: 28C16AP.A1, EEPROM_ADDR.2, SR_0A.QB
- removed net EEPROM_A10: 28C16AP.A10, SR_1A.QC
- removed net EEPROM_A2: 28C16AP.A2, EEPROM_ADDR.3, SR_0A.QC
- removed net EEPROM_A3: 28C16AP.A3, EEPROM_ADDR.4, SR_0A.QD
- removed net EEPROM_A4: 28C16AP.A4, EEPROM_ADDR.5, SR_0A.QE
- removed net EEPROM_A5: 28C16AP.A5, EEPROM_ADDR.6, SR_0A.QF
- removed net EEPROM_A6: 28C16AP.A6, EEPROM_ADDR.7, SR_0A.QG
- removed net EEPROM_A7: 28C16AP.A7, EEPROM_ADDR.8, SR_0A.QH
- removed net EEPROM_A8: 28C16AP.A8, SR_1A.QA
- removed net EEPROM_A9: 28C16AP.A9, SR_1A.QB
- removed net EEPROM_D0: 28C16AP.D0, EEPROM_DATA.1, JP_DC11_DC10.8
- removed net EEPROM_D1: 28C16AP.D1, EEPROM_DATA.2, JP_DC11_DC10.9
- removed net EEPROM_D2: 28C16AP.D2, EEPROM_DATA.3, JP_DC11_DC10.10
- removed net EEPROM_D3: 28C16AP.D3, EEPROM_DATA.4, JP_DC11_DC10.11
- removed net EEPROM_D4: 28C16AP.D4, EEPROM_DATA.5, JP_DC11_DC10.12
- removed net EEPROM_D5: 28C16AP.D5, EEPROM_DATA.6, JP_DC11_DC10.13
- removed net EEPROM_D6: 28C16AP.D6, EEPROM_DATA.7, JP_DC11_DC10.14
- removed net EEPROM_D7: 28C16AP.D7, EEPROM_DATA.8, JP_DC11_DC10.15
- removed net EEPROM_OUT_EN: 28C16AP.!OE, SR_1A.QH, WRITE_EN_LED.A
- removed net EEPROM_WRITE_EN: 28C16AP.!WE, JP_D13_VCC_GND.15, R_WRITE_EN_PU.2
- removed net N$1: POWER_LED.C, R_POWER_LED.1
- removed net N$2: R_WRITE_EN_LED.1, WRITE_EN_LED.C
- removed net N$4: SR_0A.QH*, SR_1A.SER
- removed net SR_DATA: JP_DC11_DC10.5, SR_0A.SER
- removed net SR_LATCH: JP_DC11_DC10.7, SR_0A.RCK, SR_1A.RCK
- removed net SR_SCK: JP_DC11_DC10.6, SR_0A.SCK, SR_1A.SCK
- new net A10: 28C16A_EEPROM.A10, ADDRESS.11
- new net A8: 28C16A_EEPROM.A8, ADDRESS.9
- new net A9: 28C16A_EEPROM.A9, ADDRESS.10
- new net CHIP_ENABLE: 28C16A_EEPROM.!CE, CHIP_ENABLE_TO_GND.2, ENABLE.3
- new net D0: 28C16A_EEPROM.D0, DATA.1
- new net D1: 28C16A_EEPROM.D1, DATA.2
- new net D2: 28C16A_EEPROM.D2, DATA.3
- new net D3: 28C16A_EEPROM.D3, DATA.4
- new net D4: 28C16A_EEPROM.D4, DATA.5
- new net D5: 28C16A_EEPROM.D5, DATA.6
- new net D6: 28C16A_EEPROM.D6, DATA.7
- new net D7: 28C16A_EEPROM.D7, DATA.8
- new net OUT_ENABLE: 28C16A_EEPROM.!OE, ENABLE.2
- new net WRITE_ENABLE: 28C16A_EEPROM.!WE, ENABLE.1, R_PUP_2K.2
- net A0: now also 28C16A_EEPROM.A0, ADDRESS.1; no longer JP_D13_VCC_GND.12
- net A1: now also 28C16A_EEPROM.A1, ADDRESS.2; no longer JP_D13_VCC_GND.11
- net A2: now also 28C16A_EEPROM.A2, ADDRESS.3; no longer JP_D13_VCC_GND.10
- net A3: now also 28C16A_EEPROM.A3, ADDRESS.4; no longer JP_D13_VCC_GND.9
- net A4: now also 28C16A_EEPROM.A4, ADDRESS.5; no longer JP_D13_VCC_GND.8
- net A5: now also 28C16A_EEPROM.A5, ADDRESS.6; no longer JP_D13_VCC_GND.7
- net A6: now also 28C16A_EEPROM.A6, ADDRESS.7; no longer JP_D13_VCC_GND.6
- net A7: now also 28C16A_EEPROM.A7, ADDRESS.8; no longer JP_D13_VCC_GND.5
- net GND: now also 28C16A_EEPROM.GND, CHIP_ENABLE_TO_GND.1, DATA.10; no longer 28C16AP.!CE, CAP.2, EEPROM_ADDR.10, EEPROM_DATA.10, JP_D13_VCC_GND.2, R_POWER_LED.2, R_WRITE_EN_LED.2, SR_0A.G, SR_1A.G
- net VCC: now also DATA.9, R_PUP_2K.1; no longer CAP.1, EEPROM_ADDR.9, EEPROM_DATA.9, JP_D13_VCC_GND.4, POWER_LED.A, R_WRITE_EN_PU.1, SR_0A.SCL, SR_1A.SCL
